File: plate.kicad_pcb (KiCad board)
At the start: 2 copper layers, 285.8 x 95.3 mm, 0 parts

Commit message: Fix plate to have solder mask and 3mm thick edges
Parts:
- added REF**: PinHeader_1x01_P1.00mm_Vertical, Connector_PinHeader_1.00mm:PinHeader_1x01_P1.00mm_Vertical, F.Cu at (277.4, 41.3)
Other:
- board size 285.8 x 95.3 mm -> 286.8 x 96.3 mm
Changed lines of the file:
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@@
     (tracks 1)
     (zones 0)
-    (modules 0)
+    (modules 1)
     (nets 1)
   )
@@
     (solder_mask_min_width 0.25)
     (aux_axis_origin 0 0)
-    (visible_elements FFFFFF7F)
+    (visible_elements 7FFFFFFF)
     (pcbplotparams
       (layerselection 0x010fc_ffffffff)
@@
     (uvia_drill 0.1)
   )
+  (module Connector_PinHeader_1.00mm:PinHeader_1x01_P1.00mm_Vertical (layer F.Cu)
+    (at 277.38 41.26)
+    (descr "Through hole straight pin header, 1x01, 1.00mm pitch, single row")
+    (tags "Through hole pin header THT 1x01 1.00mm single row")
+    (fp_text reference REF** (at 0 -1.56) (layer F.SilkS) hide
+      (effects (font (size 1 1) (thickness 0.15)))
+    )
+    (fp_text value PinHeader_1x01_P1.00mm_Vertical (at 0 1.56) (layer F.Fab)
+      (effects (font (size 1 1) (thickness 0.15)))
+    )
+    (fp_text user %R (at 0 0 90) (layer F.Fab)
+      (effects (font (size 0.76 0.76) (thickness 0.114)))
+    )
+    (fp_line (start 1.15 -1) (end -1.15 -1) (layer F.CrtYd) (width 0.05))
+    (fp_line (start 1.15 1) (end 1.15 -1) (layer F.CrtYd) (width 0.05))
+    (fp_line (start -1.15 1) (end 1.15 1) (layer F.CrtYd) (width 0.05))
+    (fp_line (start -1.15 -1) (end -1.15 1) (layer F.CrtYd) (width 0.05))
+    (fp_line (start -0.635 -0.1825) (end -0.3175 -0.5) (layer F.Fab) (width 0.1))
+    (fp_line (start -0.635 0.5) (end -0.635 -0.1825) (layer F.Fab) (width 0.1))
+    (fp_line (start 0.635 0.5) (end -0.635 0.5) (layer F.Fab) (width 0.1))
+    (fp_line (start 0.635 -0.5) (end 0.635 0.5) (layer F.Fab) (width 0.1))
+    (fp_line (start -0.3175 -0.5) (end 0.635 -0.5) (layer F.Fab) (width 0.1))
+    (pad 1 thru_hole circle (at -0.52 0.01) (size 0.85 0.85) (drill 0.5) (layers *.Cu *.Mask))
+    (model ${KISYS3DMOD}/Connector_PinHeader_1.00mm.3dshapes/PinHeader_1x01_P1.00mm_Vertical.wrl
+      (at (xyz 0 0 0))
+      (scale (xyz 1 1 1))
+      (rotate (xyz 0 0 0))
+    )
+  )
   (gr_line (start 138.08331 106.81968) (end 138.08331 93.81968) (layer Edge.Cuts) (width 0.2))
   (gr_line (start 152.08331 106.81968) (end 152.08331 93.81968) (layer Edge.Cuts) (width 0.2))
-  (gr_arc (start 297.864756 107.844816) (end 297.864756 109.84484) (angle -90) (layer Edge.Cuts) (width 0.2))
-  (gr_arc (start 297.864756 16.594864) (end 299.86478 16.594864) (angle -90) (layer Edge.Cuts) (width 0.2))
-  (gr_arc (start 16.114804 16.594864) (end 16.114804 14.59484) (angle -90) (layer Edge.Cuts) (width 0.2))
-  (gr_arc (start 16.114804 107.84586) (end 14.11478 107.84586) (angle -90) (layer Edge.Cuts) (width 0.2))
+  (gr_arc (start 298.37 108.349976) (end 298.37 110.35) (angle -90) (layer Edge.Cuts) (width 0.2))
+  (gr_arc (start 298.37 16.100024) (end 300.370024 16.100024) (angle -90) (layer Edge.Cuts) (width 0.2))
+  (gr_arc (start 15.610024 16.1) (end 15.610024 14.099976) (angle -90) (layer Edge.Cuts) (width 0.2))
+  (gr_arc (start 15.610024 108.35) (end 13.61 108.35) (angle -90) (layer Edge.Cuts) (width 0.2))
   (gr_line (start 257.14625 93.82) (end 257.14625 106.82) (layer Edge.Cuts) (width 0.2))
   (gr_arc (start 246.83375 93.82) (end 247.33375 93.82) (angle -90) (layer Edge.Cuts) (width 0.2))
-  (gr_line (start 14.11478 16.594864) (end 14.11478 107.84586) (layer Edge.Cuts) (width 0.2))
+  (gr_line (start 13.61 16.1) (end 13.61 108.35) (layer Edge.Cuts) (width 0.2))
   (gr_arc (start 233.83375 106.82) (end 233.33375 106.82) (angle -90) (layer Edge.Cuts) (width 0.2))
   (gr_line (start 281.45875 93.32) (end 294.45875 93.32) (layer Edge.Cuts) (width 0.2))
   (gr_line (start 233.33375 93.82) (end 233.33375 106.82) (layer Edge.Cuts) (width 0.2))
   (gr_arc (start 246.83375 106.82) (end 246.83375 107.32) (angle -90) (layer Edge.Cuts) (width 0.2))
-  (gr_line (start 299.86478 16.594864) (end 299.86478 107.844816) (layer Edge.Cuts) (width 0.2))
+  (gr_line (start 300.370024 16.100024) (end 300.370024 108.349976) (layer Edge.Cuts) (width 0.2))
   (gr_arc (start 294.45875 93.82) (end 294.95875 93.82) (angle -90) (layer Edge.Cuts) (width 0.2))
   (gr_line (start 294.95875 93.82) (end 294.95875 106.82) (layer Edge.Cuts) (width 0.2))
@@
   (gr_line (start 223.52125 93.82) (end 223.52125 106.82) (layer Edge.Cuts) (width 0.2))
   (gr_arc (start 233.83375 93.82) (end 233.83375 93.32) (angle -90) (layer Edge.Cuts) (width 0.2))
-  (gr_line (start 16.114804 14.59484) (end 297.864756 14.59484) (layer Edge.Cuts) (width 0.2))
+  (gr_line (start 15.610024 14.099976) (end 298.37 14.1) (layer Edge.Cuts) (width 0.2))
   (gr_arc (start 281.45875 93.82) (end 281.45875 93.32) (angle -90) (layer Edge.Cuts) (width 0.2))
   (gr_arc (start 270.64625 93.82) (end 271.14625 93.82) (angle -90) (layer Edge.Cuts) (width 0.2))
@@
   (gr_arc (start 257.64625 106.82) (end 257.14625 106.82) (angle -90) (layer Edge.Cuts) (width 0.2))
   (gr_arc (start 294.45875 106.82) (end 294.45875 107.32) (angle -90) (layer Edge.Cuts) (width 0.2))
-  (gr_line (start 16.114804 109.845884) (end 297.864756 109.84484) (layer Edge.Cuts) (width 0.2))
+  (gr_line (start 15.610024 110.350024) (end 298.37 110.35) (layer Edge.Cuts) (width 0.2))
   (gr_arc (start 257.64625 93.82) (end 257.64625 93.32) (angle -90) (layer Edge.Cuts) (width 0.2))
   (gr_line (start 257.64625 107.32) (end 270.64625 107.32) (layer Edge.Cuts) (width 0.2))
@@
   (gr_line (start 17.14 17.12) (end 30.139999 17.12) (layer Edge.Cuts) (width 0.2))
   (gr_line (start 16.64 17.62) (end 16.64 30.619999) (layer Edge.Cuts) (width 0.2))
-  (via (at 277.36 43.18) (size 0.8) (drill 0.4) (layers F.Cu B.Cu) (net 0))
+  (via (at 276.77 43.2) (size 0.8) (drill 0.4) (layers F.Cu B.Cu) (net 0))
 )
